File: electrical/omgkbd/omgkbd-ambient.sch (KiCad schematic (older format))
At the start: 34 parts

Commit message: Started working on connector and power
Connections:
- net +5P renamed +5V
Other:
- note added: "34 LEDS = 34 x 60mA = 2,040mA"
Changed lines of the file:
@@
 $Descr A3 16535 11693
 encoding utf-8
-Sheet 5 5
+Sheet 5 6
 Title ""
 Date "2017-11-01"
@@
 $EndComp
 Connection ~ 3625 2875
-Connection ~ 2575 1900
-$Comp
-L +5P #PWR?
-U 1 1 5A00BFE3
+Text Notes 2700 9375 0    118  ~ 0
+34 LEDS = 34 x 60mA = 2,040mA
+$Comp
+L +5V #PWR?
+U 1 1 5A03809A
 P 2575 1900
 F 0 "#PWR?" H 2575 1750 50  0001 C CNN
-F 1 "+5P" H 2590 2073 50  0000 C CNN
+F 1 "+5V" H 2590 2073 50  0000 C CNN
 F 2 "" H 2575 1900 50  0001 C CNN
 F 3 "" H 2575 1900 50  0001 C CNN
