File: electrical/omgkbd/omgkbd-backlight.sch (KiCad schematic (older format))
At the start: 61 parts

Commit message: Started working on connector and power
Connections:
- net +5P renamed +5V
Other:
- note added: "61 LEDS = 61 x 60mA = 3,660mA"
Changed lines of the file:
@@
 $Descr A4 11693 8268
 encoding utf-8
-Sheet 4 5
+Sheet 4 6
 Title "Jellyfish"
 Date "2017-11-01"
@@
 	1300 600  1750 600
 Connection ~ 1350 600
-$Comp
-L +5P #PWR?
-U 1 1 5A00CFFE
+Text Notes 950  6850 0    118  ~ 0
+61 LEDS = 61 x 60mA = 3,660mA
+$Comp
+L +5V #PWR?
+U 1 1 5A038DBB
+P 10700 6050
+F 0 "#PWR?" H 10700 5900 50  0001 C CNN
+F 1 "+5V" H 10715 6223 50  0000 C CNN
+F 2 "" H 10700 6050 50  0001 C CNN
+F 3 "" H 10700 6050 50  0001 C CNN
+	1    10700 6050
+	1    0    0    -1
+$EndComp
+$Comp
+L +5V #PWR?
+U 1 1 5A038E89
+P 10750 4875
+F 0 "#PWR?" H 10750 4725 50  0001 C CNN
+F 1 "+5V" H 10765 5048 50  0000 C CNN
+F 2 "" H 10750 4875 50  0001 C CNN
+F 3 "" H 10750 4875 50  0001 C CNN
+	1    10750 4875
+	1    0    0    -1
+$EndComp
+$Comp
+L +5V #PWR?
+U 1 1 5A038ECC
+P 10750 3750
+F 0 "#PWR?" H 10750 3600 50  0001 C CNN
+F 1 "+5V" H 10765 3923 50  0000 C CNN
+F 2 "" H 10750 3750 50  0001 C CNN
+F 3 "" H 10750 3750 50  0001 C CNN
+	1    10750 3750
+	1    0    0    -1
+$EndComp
+$Comp
+L +5V #PWR?
+U 1 1 5A039003
+P 10700 2675
+F 0 "#PWR?" H 10700 2525 50  0001 C CNN
+F 1 "+5V" H 10715 2848 50  0000 C CNN
+F 2 "" H 10700 2675 50  0001 C CNN
+F 3 "" H 10700 2675 50  0001 C CNN
+	1    10700 2675
+	1    0    0    -1
+$EndComp
+$Comp
+L +5V #PWR?
+U 1 1 5A0390FD
 P 10700 1700
 F 0 "#PWR?" H 10700 1550 50  0001 C CNN
-F 1 "+5P" H 10715 1873 50  0000 C CNN
+F 1 "+5V" H 10715 1873 50  0000 C CNN
 F 2 "" H 10700 1700 50  0001 C CNN
 F 3 "" H 10700 1700 50  0001 C CNN
@@
 $EndComp
 $Comp
-L +5P #PWR?
-U 1 1 5A00D098
-P 10700 2675
-F 0 "#PWR?" H 10700 2525 50  0001 C CNN
-F 1 "+5P" H 10715 2848 50  0000 C CNN
-F 2 "" H 10700 2675 50  0001 C CNN
-F 3 "" H 10700 2675 50  0001 C CNN
-	1    10700 2675
+L +5V #PWR?
+U 1 1 5A039328
+P 900 1700
+F 0 "#PWR?" H 900 1550 50  0001 C CNN
+F 1 "+5V" H 915 1873 50  0000 C CNN
+F 2 "" H 900 1700 50  0001 C CNN
+F 3 "" H 900 1700 50  0001 C CNN
+	1    900  1700
 	1    0    0    -1
 $EndComp
 $Comp
-L +5P #PWR?
-U 1 1 5A00D11D
-P 10750 3750
-F 0 "#PWR?" H 10750 3600 50  0001 C CNN
-F 1 "+5P" H 10765 3923 50  0000 C CNN
-F 2 "" H 10750 3750 50  0001 C CNN
-F 3 "" H 10750 3750 50  0001 C CNN
-	1    10750 3750
+L +5V #PWR?
+U 1 1 5A03936B
+P 900 2675
+F 0 "#PWR?" H 900 2525 50  0001 C CNN
+F 1 "+5V" H 915 2848 50  0000 C CNN
+F 2 "" H 900 2675 50  0001 C CNN
+F 3 "" H 900 2675 50  0001 C CNN
+	1    900  2675
 	1    0    0    -1
 $EndComp
 $Comp
-L +5P #PWR?
-U 1 1 5A00D1A2
-P 10750 4875
-F 0 "#PWR?" H 10750 4725 50  0001 C CNN
-F 1 "+5P" H 10765 5048 50  0000 C CNN
-F 2 "" H 10750 4875 50  0001 C CNN
-F 3 "" H 10750 4875 50  0001 C CNN
-	1    10750 4875
+L +5V #PWR?
+U 1 1 5A0393AE
+P 875 3750
+F 0 "#PWR?" H 875 3600 50  0001 C CNN
+F 1 "+5V" H 890 3923 50  0000 C CNN
+F 2 "" H 875 3750 50  0001 C CNN
+F 3 "" H 875 3750 50  0001 C CNN
+	1    875  3750
 	1    0    0    -1
 $EndComp
 $Comp
-L +5P #PWR?
-U 1 1 5A00D31B
-P 10700 6050
-F 0 "#PWR?" H 10700 5900 50  0001 C CNN
-F 1 "+5P" H 10715 6223 50  0000 C CNN
-F 2 "" H 10700 6050 50  0001 C CNN
-F 3 "" H 10700 6050 50  0001 C CNN
-	1    10700 6050
+L +5V #PWR?
+U 1 1 5A0394E5
+P 900 4875
+F 0 "#PWR?" H 900 4725 50  0001 C CNN
+F 1 "+5V" H 915 5048 50  0000 C CNN
+F 2 "" H 900 4875 50  0001 C CNN
+F 3 "" H 900 4875 50  0001 C CNN
+	1    900  4875
 	1    0    0    -1
 $EndComp
 $Comp
-L +5P #PWR?
-U 1 1 5A00D494
+L +5V #PWR?
+U 1 1 5A03961C
 P 900 6050
 F 0 "#PWR?" H 900 5900 50  0001 C CNN
-F 1 "+5P" H 915 6223 50  0000 C CNN
+F 1 "+5V" H 915 6223 50  0000 C CNN
 F 2 "" H 900 6050 50  0001 C CNN
 F 3 "" H 900 6050 50  0001 C CNN
@@
 	1    0    0    -1
 $EndComp
-$Comp
-L +5P #PWR?
-U 1 1 5A00D701
-P 900 4875
-F 0 "#PWR?" H 900 4725 50  0001 C CNN
-F 1 "+5P" H 915 5048 50  0000 C CNN
-F 2 "" H 900 4875 50  0001 C CNN
-F 3 "" H 900 4875 50  0001 C CNN
-	1    900  4875
-	1    0    0    -1
-$EndComp
-$Comp
-L +5P #PWR?
-U 1 1 5A00D786
-P 875 3750
-F 0 "#PWR?" H 875 3600 50  0001 C CNN
-F 1 "+5P" H 890 3923 50  0000 C CNN
-F 2 "" H 875 3750 50  0001 C CNN
-F 3 "" H 875 3750 50  0001 C CNN
-	1    875  3750
-	1    0    0    -1
-$EndComp
-$Comp
-L +5P #PWR?
-U 1 1 5A00D8FF
-P 900 2675
-F 0 "#PWR?" H 900 2525 50  0001 C CNN
-F 1 "+5P" H 915 2848 50  0000 C CNN
-F 2 "" H 900 2675 50  0001 C CNN
-F 3 "" H 900 2675 50  0001 C CNN
-	1    900  2675
-	1    0    0    -1
-$EndComp
-$Comp
-L +5P #PWR?
-U 1 1 5A00DA78
-P 900 1700
-F 0 "#PWR?" H 900 1550 50  0001 C CNN
-F 1 "+5P" H 915 1873 50  0000 C CNN
-F 2 "" H 900 1700 50  0001 C CNN
-F 3 "" H 900 1700 50  0001 C CNN
-	1    900  1700
-	1    0    0    -1
-$EndComp
